File: uae/uae.sch (KiCad schematic (older format))
At the start: 5 parts

Commit message: первая неподтвержденная версия
Parts:
- added DA2, DA3: LTV817S, N_DD:SOP-4, symbol elements:CPC1035NTR(SOP-4)
- added DA5: EDR101A0500(SIP), N_DD:реле_EDR101A0500(SIP7), symbol elements:Реле_герконовое_EDR101A0500(SIP)
- added R1, R2, R4, R6, R7: 4,7k_0,125Вт_0805, N_RLC:Резистор_SMD_0805_0,125Вт, symbol elements:Резистор_0,125Вт
- added R5: 47_0,125Вт_0805, N_RLC:Резистор_SMD_0805_0,125Вт, symbol elements:Резистор_0,125Вт
- added R8: 130_0,125Вт_0805, N_RLC:Резистор_SMD_0805_0,125Вт, symbol elements:Резистор_0,125Вт
- added VD2: S13_SOD-123, N_VD_HL:Диод_S13_SOD-123, symbol elements:Диод_шоттки
- added VT2: Транзистор_NPN_BC817-16.215, N_VD_HL:Транзистор_IRLML6344TR_SOT-23, symbol elements:Транзистор_NPN_1Б-2Э-3К
- added XP1, XP2: Вилка_PLS8, N_X:Вилка_PLS8_вертикальная, symbol elements:Вилка_PLS8
- R3: renamed from R?; value 100_0,125Вт_0805 -> 47_0,125Вт_0805
- gave numbers to parts that had none: 4
Connections:
- net labels added: 5V_OUT, COM_OUT, DI_1_RPI, DI_1_in, DI_gnd, DO_1_RPI, DO_2_RPI, GND_OUT, OUT_1, OUT_2, PULL_UP_1, PULL_UP_2, VCC_RPI
- wire segments 2 -> 77
